Commit message: Add first version of fetch mp w full motion

File: dsynth/assets/urdf/fetch/fetch.urdf (robot description, URDF)
Before this commit: robot ds_fetch, 29 links, 28 joints
Joints:
- joint root_z_rotation_joint: limit lower=-2.8973 upper=2.8973 effort=33.82 velocity=1.256 -> lower=-6.28 upper=6.28 effort=33.82 velocity=1.256; type prismatic -> revolute
