Commit message: Modified fetch with basket, mp for pick one product

File: dsynth/assets/urdf/fetch/fetch_basket.urdf (robot description, URDF)
Before this commit: robot ds_fetch, 30 links, 29 joints
Links:
- added link basket002; collision mesh filename=fetch_description/meshes/basket002.obj; visual mesh filename=fetch_description/meshes/basket002.obj
- added link basket003; collision mesh filename=fetch_description/meshes/basket003.obj; visual mesh filename=fetch_description/meshes/basket003.obj
- added link basket004; collision mesh filename=fetch_description/meshes/basket004.obj; visual mesh filename=fetch_description/meshes/basket004.obj
- added link basket005; collision mesh filename=fetch_description/meshes/basket005.obj; visual mesh filename=fetch_description/meshes/basket005.obj
- added link basket006; collision mesh filename=fetch_description/meshes/basket006.obj; visual mesh filename=fetch_description/meshes/basket006.obj
- added link basket007; collision mesh filename=fetch_description/meshes/basket007.obj; visual mesh filename=fetch_description/meshes/basket007.obj
- added link basket008; collision mesh filename=fetch_description/meshes/basket008.obj; visual mesh filename=fetch_description/meshes/basket008.obj
- added link basket009; collision mesh filename=fetch_description/meshes/basket009.obj; visual mesh filename=fetch_description/meshes/basket009.obj
Joints:
- removed joint basket_joint
- added joint basket002: type fixed, parent basket, child basket002, origin xyz=0 0 0 rpy=0 0 0, axis 0 1 0
- added joint basket003: type fixed, parent basket, child basket003, origin xyz=0 0 0 rpy=0 0 0, axis 0 1 0
- added joint basket004: type fixed, parent basket, child basket004, origin xyz=0 0 0 rpy=0 0 0, axis 0 1 0
- added joint basket005: type fixed, parent basket, child basket005, origin xyz=0 0 0 rpy=0 0 0, axis 0 1 0
- added joint basket006: type fixed, parent basket, child basket006, origin xyz=0 0 0 rpy=0 0 0, axis 0 1 0
- added joint basket007: type fixed, parent basket, child basket007, origin xyz=0 0 0 rpy=0 0 0, axis 0 1 0
- added joint basket008: type fixed, parent basket, child basket008, origin xyz=0 0 0 rpy=0 0 0, axis 0 1 0
- added joint basket009: type fixed, parent basket, child basket009, origin xyz=0 0 0 rpy=0 0 0, axis 0 1 0
- added joint basket_joint_base: type fixed, parent base_link, child basket, origin xyz=0 0 0 rpy=0 0 0, axis 0 1 0

Commit message: Removed unused joints in fetch_basket

File: dsynth/assets/urdf/fetch/fetch_basket.urdf (robot description, URDF)
Before this commit: robot ds_fetch, 38 links, 37 joints
Links:
- removed link basket002
- removed link basket003
- removed link basket004
- removed link basket005
- removed link basket006
- removed link basket007
- removed link basket008
- removed link basket009
- link basket: geometry collision mesh filename=fetch_description/meshes/basket.obj; collision mesh filename=fetch_description/meshes/basket002.obj
Joints:
- removed joint basket002
- removed joint basket003
- removed joint basket004
- removed joint basket005
- removed joint basket006
- removed joint basket007
- removed joint basket008
- removed joint basket009
