Commit message: Add fetch_basket_static

File: dsynth/assets/urdf/fetch/fetch_basket_static.urdf (robot description, URDF)
Before this commit: robot ds_fetch_basket, 30 links, 29 joints
Joints:
- joint root_x_axis_joint: type prismatic -> fixed
- joint root_y_axis_joint: type prismatic -> fixed
- joint root_z_rotation_joint: type revolute -> fixed
